File: ESP8266Tetris.kicad_pcb (KiCad board)
At the start: 2 copper layers, 60 x 120 mm, 235 parts, among them J1 10118192-0001LF, Q1 BC847BLT1G, Q2 DMP3068L-7, Q3 BC847BLT1G, Q4 BC847BLT1G, Q5 BC847BLT1G, Q6 DMP3068L-7, Q7 BC847BLT1G, Q8 BC847BLT1G, Q9 BC847BLT1G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

Commit message: Buttons debounce capacitors value changed from 10n to 220n.
Signed-off-by: Ion Bold <bold.ion86@gmail.com>
Parts:
- C12, C13, C14, C15, C16: value 10n -> 220n
Changed lines of the file:
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@@
       (effects (font (size 1 1) (thickness 0.15)))
     )
-    (fp_text value "10n" (at 0 1.43 45) (layer "F.Fab")
+    (fp_text value "220n" (at 0 1.43 45) (layer "F.Fab")
       (effects (font (size 1 1) (thickness 0.15)))
     )
@@
       (effects (font (size 1 1) (thickness 0.15)))
     )
-    (fp_text value "10n" (at 0 1.43 45) (layer "F.Fab")
+    (fp_text value "220n" (at 0 1.43 45) (layer "F.Fab")
       (effects (font (size 1 1) (thickness 0.15)))
     )
@@
       (effects (font (size 1 1) (thickness 0.15)))
     )
-    (fp_text value "10n" (at 0 1.43 45) (layer "F.Fab")
+    (fp_text value "220n" (at 0 1.43 45) (layer "F.Fab")
       (effects (font (size 1 1) (thickness 0.15)))
     )
@@
       (effects (font (size 1 1) (thickness 0.15)))
     )
-    (fp_text value "10n" (at 0 1.43 45) (layer "F.Fab")
+    (fp_text value "220n" (at 0 1.43 45) (layer "F.Fab")
       (effects (font (size 1 1) (thickness 0.15)))
     )
@@
       (effects (font (size 1 1) (thickness 0.15)))
     )
-    (fp_text value "10n" (at 0 1.43 45) (layer "F.Fab")
+    (fp_text value "220n" (at 0 1.43 45) (layer "F.Fab")
       (effects (font (size 1 1) (thickness 0.15)))
     )
