File: ESP8266Tetris.kicad_sch (KiCad schematic)
At the start: 84 parts, among them J1 10118192-0001LF, Q1 BC847BLT1G, Q2 DMP3068L-7, Q3 BC847BLT1G, Q4 BC847BLT1G, Q5 BC847BLT1G, Q6 DMP3068L-7, Q7 BC847BLT1G, Q8 BC847BLT1G, Q9 BC847BLT1G, SW1 B3AL-1006P, SW2 B3AL-1006P, SW3 B3AL-1006P, SW4 B3AL-1006P, SW5 B3AL-1006P, SW6 B3AL-1006P, U1 CH340G, U2 ESP-12F, U3 BQ25170DSGR, U4 LP3874EMPX-3.3/NOPB, Y1 ABM3-12.000MHZ-D2Y-T

Commit message: Routing PCB done.
Signed-off-by: Ion Bold <bold.ion86@gmail.com>
Parts:
- Y1: footprint Crystal:Crystal_SMD_7050-2Pin_7.0x5.0mm_HandSoldering -> Crystal:Crystal_SMD_7050-2Pin_7.0x5.0mm
Other:
- note removed: "TODO: - verificat configuratie pini DOUT si BUZZER cf. datasheet - verificat functionare GPIO2, GPIO15, GPIO16 pe breadboard - verificat butoane cu pull-up si pull-down extern pe breadboard"
Changed lines of the file:
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@@
     (effects (font (size 1 1)) (justify left bottom))
   )
-  (text "TODO:\n- verificat configuratie pini DOUT si BUZZER cf. datasheet\n- verificat functionare GPIO2, GPIO15, GPIO16 pe breadboard\n- verificat butoane cu pull-up si pull-down extern pe breadboard"
-    (at 137.16 124.46 0)
-    (effects (font (size 1.27 1.27) bold italic) (justify left bottom))
-  )
   (text "10u / 16V" (at 154.305 60.325 0)
     (effects (font (size 1.27 1.27)) (justify left bottom))
@@
       (effects (font (size 1 1)))
     )
-    (property "Footprint" "Crystal:Crystal_SMD_7050-2Pin_7.0x5.0mm_HandSoldering" (id 2) (at 34.29 177.8 0)
+    (property "Footprint" "Crystal:Crystal_SMD_7050-2Pin_7.0x5.0mm" (id 2) (at 34.29 177.8 0)
       (effects (font (size 1.27 1.27)) hide)
     )
@@
     )
     (path "/ef739389-f27b-461c-8d68-f13f7571f72f"
-      (reference "Y1") (unit 1) (value "ABM3-12.000MHZ-D2Y-T") (footprint "Crystal:Crystal_SMD_7050-2Pin_7.0x5.0mm_HandSoldering")
+      (reference "Y1") (unit 1) (value "ABM3-12.000MHZ-D2Y-T") (footprint "Crystal:Crystal_SMD_7050-2Pin_7.0x5.0mm")
     )
   )

Commit message: Fabrication and assembly files generated (v1.0).
Signed-off-by: Ion Bold <bold.ion86@gmail.com>
Parts:
- added H5, H6, H7, H8: Hole, MountingHole:MountingHole_2.2mm_M2, symbol Mechanical:MountingHole
- C11, C33, C34, C35, C9: footprint Capacitor_Tantalum_SMD:CP_EIA-3216-12_Kemet-S_Pad1.58x1.35mm_HandSolder -> Capacitor_Tantalum_SMD:CP_EIA-3216-18_Kemet-A_Pad1.58x1.35mm_HandSolder
- H1, H2, H3, H4: now left out of the parts list
Changed lines of the file:
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@@
       (effects (font (size 1.27 1.27)) (justify left))
     )
-    (property "Footprint" "Capacitor_Tantalum_SMD:CP_EIA-3216-12_Kemet-S_Pad1.58x1.35mm_HandSolder" (id 2) (at 255.27 46.99 0)
+    (property "Footprint" "Capacitor_Tantalum_SMD:CP_EIA-3216-18_Kemet-A_Pad1.58x1.35mm_HandSolder" (id 2) (at 255.27 46.99 0)
       (effects (font (size 1.27 1.27)) hide)
     )
@@
       (effects (font (size 1.27 1.27)) (justify left))
     )
-    (property "Footprint" "Capacitor_Tantalum_SMD:CP_EIA-3216-12_Kemet-S_Pad1.58x1.35mm_HandSolder" (id 2) (at 152.4 54.61 0)
+    (property "Footprint" "Capacitor_Tantalum_SMD:CP_EIA-3216-18_Kemet-A_Pad1.58x1.35mm_HandSolder" (id 2) (at 152.4 54.61 0)
       (effects (font (size 1.27 1.27)) hide)
     )
@@
   )
   (symbol (lib_id "Mechanical:MountingHole_Pad") (at 160.02 29.21 0) (unit 1)
-    (in_bom yes) (on_board yes)
+    (in_bom no) (on_board yes)
     (property "Reference" "H3" (id 0) (at 161.29 25.4 0)
       (effects (font (size 1.27 1.27)) (justify left))
@@
     (pin "1")
   )
+  (symbol (lib_id "Mechanical:MountingHole") (at 158.75 175.26 0) (unit 1)
+    (in_bom no) (on_board yes) (fields_autoplaced)
+    (property "Reference" "H7" (id 0) (at 161.29 173.9899 0)
+      (effects (font (size 1.27 1.27)) (justify left))
+    )
+    (property "Value" "Hole" (id 1) (at 161.29 176.5299 0)
+      (effects (font (size 1.27 1.27)) (justify left))
+    )
+    (property "Footprint" "MountingHole:MountingHole_2.2mm_M2" (id 2) (at 158.75 175.26 0)
+      (effects (font (size 1.27 1.27)) hide)
+    )
+    (property "Datasheet" "~" (id 3) (at 158.75 175.26 0)
+      (effects (font (size 1.27 1.27)) hide)
+    )
+  )
   (symbol (lib_id "power:GND") (at 52.07 186.69 0) (unit 1)
     (in_bom yes) (on_board yes)
@@
   )
   (symbol (lib_id "Mechanical:MountingHole_Pad") (at 153.67 29.21 0) (unit 1)
-    (in_bom yes) (on_board yes)
+    (in_bom no) (on_board yes)
     (property "Reference" "H2" (id 0) (at 154.94 25.4 0)
       (effects (font (size 1.27 1.27)) (justify left))
@@
       (effects (font (size 1.27 1.27)) (justify left))
     )
-    (property "Footprint" "Capacitor_Tantalum_SMD:CP_EIA-3216-12_Kemet-S_Pad1.58x1.35mm_HandSolder" (id 2) (at 182.88 54.61 0)
+    (property "Footprint" "Capacitor_Tantalum_SMD:CP_EIA-3216-18_Kemet-A_Pad1.58x1.35mm_HandSolder" (id 2) (at 182.88 54.61 0)
       (effects (font (size 1.27 1.27)) hide)
     )
@@
     (pin "1")
   )
+  (symbol (lib_id "Mechanical:MountingHole") (at 147.32 175.26 0) (unit 1)
+    (in_bom no) (on_board yes) (fields_autoplaced)
+    (property "Reference" "H5" (id 0) (at 149.86 173.9899 0)
+      (effects (font (size 1.27 1.27)) (justify left))
+    )
+    (property "Value" "Hole" (id 1) (at 149.86 176.5299 0)
+      (effects (font (size 1.27 1.27)) (justify left))
+    )
+    (property "Footprint" "MountingHole:MountingHole_2.2mm_M2" (id 2) (at 147.32 175.26 0)
+      (effects (font (size 1.27 1.27)) hide)
+    )
+    (property "Datasheet" "~" (id 3) (at 147.32 175.26 0)
+      (effects (font (size 1.27 1.27)) hide)
+    )
+  )
   (symbol (lib_id "Device:C_Small") (at 39.37 182.88 0) (unit 1)
     (in_bom yes) (on_board yes)
@@
     (pin "3")
   )
+  (symbol (lib_id "Mechanical:MountingHole") (at 158.75 184.15 0) (unit 1)
+    (in_bom no) (on_board yes) (fields_autoplaced)
+    (property "Reference" "H8" (id 0) (at 161.29 182.8799 0)
+      (effects (font (size 1.27 1.27)) (justify left))
+    )
+    (property "Value" "Hole" (id 1) (at 161.29 185.4199 0)
+      (effects (font (size 1.27 1.27)) (justify left))
+    )
+    (property "Footprint" "MountingHole:MountingHole_2.2mm_M2" (id 2) (at 158.75 184.15 0)
+      (effects (font (size 1.27 1.27)) hide)
+    )
+    (property "Datasheet" "~" (id 3) (at 158.75 184.15 0)
+      (effects (font (size 1.27 1.27)) hide)
+    )
+  )
   (symbol (lib_id "Device:C_Small") (at 240.03 99.06 0) (mirror y) (unit 1)
     (in_bom yes) (on_board yes)
@@
       (effects (font (size 1.27 1.27)) (justify left))
     )
-    (property "Footprint" "Capacitor_Tantalum_SMD:CP_EIA-3216-12_Kemet-S_Pad1.58x1.35mm_HandSolder" (id 2) (at 238.76 46.99 0)
+    (property "Footprint" "Capacitor_Tantalum_SMD:CP_EIA-3216-18_Kemet-A_Pad1.58x1.35mm_HandSolder" (id 2) (at 238.76 46.99 0)
       (effects (font (size 1.27 1.27)) hide)
     )
@@
       (effects (font (size 1.27 1.27)) (justify left))
     )
-    (property "Footprint" "Capacitor_Tantalum_SMD:CP_EIA-3216-12_Kemet-S_Pad1.58x1.35mm_HandSolder" (id 2) (at 246.38 46.99 0)
+    (property "Footprint" "Capacitor_Tantalum_SMD:CP_EIA-3216-18_Kemet-A_Pad1.58x1.35mm_HandSolder" (id 2) (at 246.38 46.99 0)
       (effects (font (size 1.27 1.27)) hide)
     )
@@
     (pin "1")
   )
+  (symbol (lib_id "Mechanical:MountingHole") (at 147.32 184.15 0) (unit 1)
+    (in_bom no) (on_board yes) (fields_autoplaced)
+    (property "Reference" "H6" (id 0) (at 149.86 182.8799 0)
+      (effects (font (size 1.27 1.27)) (justify left))
+    )
+    (property "Value" "Hole" (id 1) (at 149.86 185.4199 0)
+      (effects (font (size 1.27 1.27)) (justify left))
+    )
+    (property "Footprint" "MountingHole:MountingHole_2.2mm_M2" (id 2) (at 147.32 184.15 0)
+      (effects (font (size 1.27 1.27)) hide)
+    )
+    (property "Datasheet" "~" (id 3) (at 147.32 184.15 0)
+      (effects (font (size 1.27 1.27)) hide)
+    )
+  )
   (symbol (lib_id "power:+3V3") (at 24.13 74.93 0) (unit 1)
     (in_bom yes) (on_board yes)
@@
   )
   (symbol (lib_id "Mechanical:MountingHole_Pad") (at 147.32 29.21 0) (unit 1)
-    (in_bom yes) (on_board yes)
+    (in_bom no) (on_board yes)
     (property "Reference" "H1" (id 0) (at 148.59 25.4 0)
       (effects (font (size 1.27 1.27)) (justify left))
@@
   )
   (symbol (lib_id "Mechanical:MountingHole_Pad") (at 166.37 29.21 0) (unit 1)
-    (in_bom yes) (on_board yes)
+    (in_bom no) (on_board yes)
     (property "Reference" "H4" (id 0) (at 167.64 25.4 0)
       (effects (font (size 1.27 1.27)) (justify left))
@@
     )
     (path "/45a7e6e3-63cd-457d-8e82-fd516ea6e35c"
-      (reference "C9") (unit 1) (value "TAJA106K016RNJ") (footprint "Capacitor_Tantalum_SMD:CP_EIA-3216-12_Kemet-S_Pad1.58x1.35mm_HandSolder")
+      (reference "C9") (unit 1) (value "TAJA106K016RNJ") (footprint "Capacitor_Tantalum_SMD:CP_EIA-3216-18_Kemet-A_Pad1.58x1.35mm_HandSolder")
     )
     (path "/360a11ab-93df-4177-b908-3f60549b35a0"
@@
     )
     (path "/7640a33e-49dc-4fa9-bf36-c02a3d43528b"
-      (reference "C11") (unit 1) (value "TAJA106K016RNJ") (footprint "Capacitor_Tantalum_SMD:CP_EIA-3216-12_Kemet-S_Pad1.58x1.35mm_HandSolder")
+      (reference "C11") (unit 1) (value "TAJA106K016RNJ") (footprint "Capacitor_Tantalum_SMD:CP_EIA-3216-18_Kemet-A_Pad1.58x1.35mm_HandSolder")
     )
     (path "/a03508f5-441c-4d0b-9396-950a58bda1da"
@@
     )
     (path "/b55be60f-d393-4c77-9e0a-04df8a2e00d7"
-      (reference "C33") (unit 1) (value "TAJA106K016RNJ") (footprint "Capacitor_Tantalum_SMD:CP_EIA-3216-12_Kemet-S_Pad1.58x1.35mm_HandSolder")
+      (reference "C33") (unit 1) (value "TAJA106K016RNJ") (footprint "Capacitor_Tantalum_SMD:CP_EIA-3216-18_Kemet-A_Pad1.58x1.35mm_HandSolder")
     )
     (path "/d6234140-6eb6-42cc-b3da-a90e7eaa6b3b"
-      (reference "C34") (unit 1) (value "TAJA106K016RNJ") (footprint "Capacitor_Tantalum_SMD:CP_EIA-3216-12_Kemet-S_Pad1.58x1.35mm_HandSolder")
+      (reference "C34") (unit 1) (value "TAJA106K016RNJ") (footprint "Capacitor_Tantalum_SMD:CP_EIA-3216-18_Kemet-A_Pad1.58x1.35mm_HandSolder")
     )
     (path "/15359d16-2525-4b4f-b619-988dd237935f"
-      (reference "C35") (unit 1) (value "TAJA106K016RNJ") (footprint "Capacitor_Tantalum_SMD:CP_EIA-3216-12_Kemet-S_Pad1.58x1.35mm_HandSolder")
+      (reference "C35") (unit 1) (value "TAJA106K016RNJ") (footprint "Capacitor_Tantalum_SMD:CP_EIA-3216-18_Kemet-A_Pad1.58x1.35mm_HandSolder")
     )
     (path "/ec8e3ae1-2f31-424b-8995-60aa9b815076"
@@
       (reference "H4") (unit 1) (value "MH") (footprint "MountingHole:MountingHole_3.2mm_M3_DIN965_Pad")
     )
+    (path "/8857114d-9688-4ebf-bf44-ca6a7b8be959"
+      (reference "H5") (unit 1) (value "Hole") (footprint "MountingHole:MountingHole_2.2mm_M2")
+    )
+    (path "/d7e32b15-bdf4-48c0-a1f6-b4b1d0844209"
+      (reference "H6") (unit 1) (value "Hole") (footprint "MountingHole:MountingHole_2.2mm_M2")
+    )
+    (path "/6870c09f-3447-454c-a0ae-4a923da25444"
+      (reference "H7") (unit 1) (value "Hole") (footprint "MountingHole:MountingHole_2.2mm_M2")
+    )
+    (path "/9b064e11-74f1-4c68-a555-deefb937ab2f"
+      (reference "H8") (unit 1) (value "Hole") (footprint "MountingHole:MountingHole_2.2mm_M2")
+    )
     (path "/5573d225-e7b9-4d29-bac0-9475e3c7e748"

Commit message: Buttons debounce capacitors value changed from 10n to 220n.
Signed-off-by: Ion Bold <bold.ion86@gmail.com>
Parts:
- C12, C13, C14, C15, C16: value 10n -> 220n
Changed lines of the file:
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@@
       (effects (font (size 1.27 1.27)) (justify left))
     )
-    (property "Value" "10n" (id 1) (at 213.36 101.6 0)
+    (property "Value" "220n" (id 1) (at 213.36 101.6 0)
       (effects (font (size 1.27 1.27)) (justify left))
     )
@@
       (effects (font (size 1.27 1.27)) (justify left))
     )
-    (property "Value" "10n" (id 1) (at 167.64 101.6 0)
+    (property "Value" "220n" (id 1) (at 167.64 101.6 0)
       (effects (font (size 1.27 1.27)) (justify left))
     )
@@
       (effects (font (size 1.27 1.27)) (justify left))
     )
-    (property "Value" "10n" (id 1) (at 238.76 101.6 0)
+    (property "Value" "220n" (id 1) (at 238.76 101.6 0)
       (effects (font (size 1.27 1.27)) (justify left))
     )
@@
       (effects (font (size 1.27 1.27)) (justify left))
     )
-    (property "Value" "10n" (id 1) (at 146.05 101.6 0)
+    (property "Value" "220n" (id 1) (at 146.05 101.6 0)
       (effects (font (size 1.27 1.27)) (justify left))
     )
@@
       (effects (font (size 1.27 1.27)) (justify left))
     )
-    (property "Value" "10n" (id 1) (at 190.5 101.6 0)
+    (property "Value" "220n" (id 1) (at 190.5 101.6 0)
       (effects (font (size 1.27 1.27)) (justify left))
     )
@@
     )
     (path "/a03508f5-441c-4d0b-9396-950a58bda1da"
-      (reference "C12") (unit 1) (value "10n") (footprint "Capacitor_SMD:C_0603_1608Metric_Pad1.08x0.95mm_HandSolder")
+      (reference "C12") (unit 1) (value "220n") (footprint "Capacitor_SMD:C_0603_1608Metric_Pad1.08x0.95mm_HandSolder")
     )
     (path "/748cecf3-200c-465a-a043-70698a891c7f"
-      (reference "C13") (unit 1) (value "10n") (footprint "Capacitor_SMD:C_0603_1608Metric_Pad1.08x0.95mm_HandSolder")
+      (reference "C13") (unit 1) (value "220n") (footprint "Capacitor_SMD:C_0603_1608Metric_Pad1.08x0.95mm_HandSolder")
     )
     (path "/f2bfa29f-6304-4137-9a10-95548cf9fb8b"
-      (reference "C14") (unit 1) (value "10n") (footprint "Capacitor_SMD:C_0603_1608Metric_Pad1.08x0.95mm_HandSolder")
+      (reference "C14") (unit 1) (value "220n") (footprint "Capacitor_SMD:C_0603_1608Metric_Pad1.08x0.95mm_HandSolder")
     )
     (path "/3863adc1-18e4-4e35-b809-951092e8fc1e"
-      (reference "C15") (unit 1) (value "10n") (footprint "Capacitor_SMD:C_0603_1608Metric_Pad1.08x0.95mm_HandSolder")
+      (reference "C15") (unit 1) (value "220n") (footprint "Capacitor_SMD:C_0603_1608Metric_Pad1.08x0.95mm_HandSolder")
     )
     (path "/9b417f1e-c79c-48c6-b3a2-bb9b8ff63ca5"
-      (reference "C16") (unit 1) (value "10n") (footprint "Capacitor_SMD:C_0603_1608Metric_Pad1.08x0.95mm_HandSolder")
+      (reference "C16") (unit 1) (value "220n") (footprint "Capacitor_SMD:C_0603_1608Metric_Pad1.08x0.95mm_HandSolder")
     )
     (path "/3bb43f88-3289-4ebd-9acf-9a6fde136db1/526bb787-22dc-4a72-b5c9-1995b3925789"
